Commit message: <urdf>: switch from .dae to .stl

File: resources/robots/go1/urdf/go1.urdf (robot description, URDF)
Before this commit: robot go1, 34 links, 33 joints
Links:
- removed link camera_chin
- removed link camera_face
- removed link camera_laserscan_link_left
- removed link camera_laserscan_link_right
- removed link camera_left
- removed link camera_optical_chin
- removed link camera_optical_face
- removed link camera_optical_left
- removed link camera_optical_rearDown
- removed link camera_optical_right
- removed link camera_rearDown
- removed link camera_right
- removed link ultraSound_face
- removed link ultraSound_left
- removed link ultraSound_right
- link FL_calf: geometry collision box size=0.213 0.016 0.016; visual mesh filename=../meshes/calf.stl scale=1 1 1
- link FL_hip: geometry collision cylinder length=0.04 radius=0.046; visual mesh filename=../meshes/hip.stl scale=1 1 1
- link FL_thigh: geometry collision box size=0.213 0.0245 0.034; visual mesh filename=../meshes/thigh.stl scale=1 1 1
- link FR_calf: geometry collision box size=0.213 0.016 0.016; visual mesh filename=../meshes/calf.stl scale=1 1 1
- link FR_hip: geometry collision cylinder length=0.04 radius=0.046; visual mesh filename=../meshes/hip.stl scale=1 1 1
- link FR_thigh: geometry collision box size=0.213 0.0245 0.034; visual mesh filename=../meshes/thigh_mirror.stl scale=1 1 1
- link RL_calf: geometry collision box size=0.213 0.016 0.016; visual mesh filename=../meshes/calf.stl scale=1 1 1
- link RL_hip: geometry collision cylinder length=0.04 radius=0.046; visual mesh filename=../meshes/hip.stl scale=1 1 1
- link RL_thigh: geometry collision box size=0.213 0.0245 0.034; visual mesh filename=../meshes/thigh.stl scale=1 1 1
- link RR_calf: geometry collision box size=0.213 0.016 0.016; visual mesh filename=../meshes/calf.stl scale=1 1 1
- link RR_hip: geometry collision cylinder length=0.04 radius=0.046; visual mesh filename=../meshes/hip.stl scale=1 1 1
- link RR_thigh: geometry collision box size=0.213 0.0245 0.034; visual mesh filename=../meshes/thigh_mirror.stl scale=1 1 1
- link trunk: geometry collision box size=0.3762 0.0935 0.114; visual mesh filename=../meshes/trunk.stl scale=1 1 1
Joints:
- removed joint camera_joint_chin
- removed joint camera_joint_face
- removed joint camera_joint_left
- removed joint camera_joint_rearDown
- removed joint camera_joint_right
- removed joint camera_laserscan_joint_left
- removed joint camera_laserscan_joint_right
- removed joint camera_optical_joint_chin
- removed joint camera_optical_joint_face
- removed joint camera_optical_joint_left
- removed joint camera_optical_joint_rearDown
- removed joint camera_optical_joint_right
- removed joint ultraSound_joint_face
- removed joint ultraSound_joint_left
- removed joint ultraSound_joint_right

File: resources/robots/go1/urdf/go1_roller.urdf (robot description, URDF)
Before this commit: robot go1, 34 links, 33 joints
Links:
- removed link camera_chin
- removed link camera_face
- removed link camera_laserscan_link_left
- removed link camera_laserscan_link_right
- removed link camera_left
- removed link camera_optical_chin
- removed link camera_optical_face
- removed link camera_optical_left
- removed link camera_optical_rearDown
- removed link camera_optical_right
- removed link camera_rearDown
- removed link camera_right
- removed link ultraSound_face
- removed link ultraSound_left
- removed link ultraSound_right
- link FL_calf: geometry collision box size=0.213 0.016 0.016; visual mesh filename=../meshes/calf.stl scale=1 1 1
- link FL_hip: geometry collision cylinder length=0.04 radius=0.046; visual mesh filename=../meshes/hip.stl scale=1 1 1
- link FL_thigh: geometry collision box size=0.213 0.0245 0.034; visual mesh filename=../meshes/thigh.stl scale=1 1 1
- link FR_calf: geometry collision box size=0.213 0.016 0.016; visual mesh filename=../meshes/calf.stl scale=1 1 1
- link FR_hip: geometry collision cylinder length=0.04 radius=0.046; visual mesh filename=../meshes/hip.stl scale=1 1 1
- link FR_thigh: geometry collision box size=0.213 0.0245 0.034; visual mesh filename=../meshes/thigh_mirror.stl scale=1 1 1
- link RL_calf: geometry collision box size=0.213 0.016 0.016; visual mesh filename=../meshes/calf.stl scale=1 1 1
- link RL_hip: geometry collision cylinder length=0.04 radius=0.046; visual mesh filename=../meshes/hip.stl scale=1 1 1
- link RL_thigh: geometry collision box size=0.213 0.0245 0.034; visual mesh filename=../meshes/thigh.stl scale=1 1 1
- link RR_calf: geometry collision box size=0.213 0.016 0.016; visual mesh filename=../meshes/calf.stl scale=1 1 1
- link RR_hip: geometry collision cylinder length=0.04 radius=0.046; visual mesh filename=../meshes/hip.stl scale=1 1 1
- link RR_thigh: geometry collision box size=0.213 0.0245 0.034; visual mesh filename=../meshes/thigh_mirror.stl scale=1 1 1
- link trunk: geometry collision box size=0.3762 0.0935 0.114; visual mesh filename=../meshes/trunk.stl scale=1 1 1
Joints:
- removed joint camera_joint_chin
- removed joint camera_joint_face
- removed joint camera_joint_left
- removed joint camera_joint_rearDown
- removed joint camera_joint_right
- removed joint camera_laserscan_joint_left
- removed joint camera_laserscan_joint_right
- removed joint camera_optical_joint_chin
- removed joint camera_optical_joint_face
- removed joint camera_optical_joint_left
- removed joint camera_optical_joint_rearDown
- removed joint camera_optical_joint_right
- removed joint ultraSound_joint_face
- removed joint ultraSound_joint_left
- removed joint ultraSound_joint_right
- joint FL_roller_hinge: origin xyz=-0.02 0 -0.243 rpy=0 0 0 -> xyz=-0.032 0 -0.25 rpy=0 0 0; type continuous -> revolute
- joint FR_roller_hinge: origin xyz=-0.02 0 -0.243 rpy=0 0 0 -> xyz=-0.032 0 -0.25 rpy=0 0 0; type continuous -> revolute
- joint RL_roller_hinge: origin xyz=-0.02 0 -0.243 rpy=0 0 0 -> xyz=-0.032 0 -0.25 rpy=0 0 0; type continuous -> revolute
- joint RR_roller_hinge: origin xyz=-0.02 0 -0.243 rpy=0 0 0 -> xyz=-0.032 0 -0.25 rpy=0 0 0; type continuous -> revolute
