Commit message: <go1_flat_roller>: split roller into v & x configuration

File: resources/robots/go1/urdf/go1_roller_v.urdf (robot description, URDF)
Before this commit: robot go1, 19 links, 18 joints
Joints:
- joint FL_roller_hinge: origin xyz=-0.032 0 -0.25 rpy=0 0 0 -> xyz=-0.032 0 -0.25 rpy=0 0 0.524
- joint FR_roller_hinge: origin xyz=-0.032 0 -0.25 rpy=0 0 0 -> xyz=-0.032 0 -0.25 rpy=0 0 -0.524
- joint RL_roller_hinge: origin xyz=-0.032 0 -0.25 rpy=0 0 0 -> xyz=-0.032 0 -0.25 rpy=0 0 0.524
- joint RR_roller_hinge: origin xyz=-0.032 0 -0.25 rpy=0 0 0 -> xyz=-0.032 0 -0.25 rpy=0 0 -0.524
